Commit message: update go2w

File: source/robot_lab/data/Robots/Unitree/Go2W/urdf/go2w_description/urdf/go2w_description.urdf (robot description, URDF)
Before this commit: robot go2w_description, 31 links, 30 joints
Links:
- added link imu, mass 0
- added link radar, mass 0
- link FL_calf: geometry collision cylinder length=0.12 radius=0.012; visual mesh filename=package://go2w_description/dae/calf.stl
- link FL_foot: geometry collision mesh filename=package://go2w_description/dae/left_wheel.dae; visual mesh filename=package://go2w_description/dae/left_wheel.dae
- link FL_hip: geometry collision cylinder length=0.04 radius=0.046; visual mesh filename=package://go2w_description/dae/hip.dae
- link FL_thigh: geometry collision box size=0.11 0.0245 0.034; visual mesh filename=package://go2w_description/dae/thigh.dae
- link FR_calf: geometry collision cylinder length=0.12 radius=0.013; visual mesh filename=package://go2w_description/dae/calf_mirror.stl
- link FR_foot: geometry collision mesh filename=package://go2w_description/dae/right_wheel.dae; visual mesh filename=package://go2w_description/dae/right_wheel.dae
- link FR_hip: geometry collision cylinder length=0.04 radius=0.046; visual mesh filename=package://go2w_description/dae/hip.dae
- link FR_thigh: geometry collision box size=0.11 0.0245 0.034; visual mesh filename=package://go2w_description/dae/thigh_mirror.dae
- link RL_calf: geometry collision cylinder length=0.12 radius=0.013; visual mesh filename=package://go2w_description/dae/calf.stl
- link RL_foot: geometry collision mesh filename=package://go2w_description/dae/left_wheel.dae; visual mesh filename=package://go2w_description/dae/left_wheel.dae
- link RL_hip: geometry collision cylinder length=0.04 radius=0.046; visual mesh filename=package://go2w_description/dae/hip.dae
- link RL_thigh: geometry collision box size=0.11 0.0245 0.034; visual mesh filename=package://go2w_description/dae/thigh.dae
- link RR_calf: geometry collision cylinder length=0.12 radius=0.013; visual mesh filename=package://go2w_description/dae/calf_mirror.stl
- link RR_foot: geometry collision mesh filename=package://go2w_description/dae/right_wheel.dae; visual mesh filename=package://go2w_description/dae/right_wheel.dae
- link RR_hip: geometry collision cylinder length=0.04 radius=0.046; visual mesh filename=package://go2w_description/dae/hip.dae
- link RR_thigh: geometry collision box size=0.11 0.0245 0.034; visual mesh filename=package://go2w_description/dae/thigh_mirror.dae
- link base: geometry collision box size=0.3762 0.0935 0.114; visual mesh filename=package://go2w_description/dae/base.dae
Joints:
- added joint imu_joint: type fixed, parent base, child imu, origin xyz=-0.02557 0 0.04232 rpy=0 0 0, axis 0 0 0
- added joint radar_joint: type fixed, parent base, child radar, origin xyz=0.28945 0 -0.046825 rpy=0 2.8782 0, axis 0 0 0

Commit message: go2w

File: source/robot_lab/data/Robots/Unitree/Go2W/urdf/go2w_description/urdf/go2w_description.urdf (robot description, URDF)
Before this commit: robot go2w_description, 33 links, 32 joints
Links:
- link FL_calf: geometry collision cylinder length=0.12 radius=0.012; visual mesh filename=package://go2w_description/dae/calf.dae
- link FL_foot: geometry collision cylinder length=0.045 radius=0.086; visual mesh filename=package://go2w_description/dae/left_wheel.dae
- link FR_calf: geometry collision cylinder length=0.12 radius=0.013; visual mesh filename=package://go2w_description/dae/calf_mirror.dae
- link FR_foot: geometry collision cylinder length=0.045 radius=0.086; visual mesh filename=package://go2w_description/dae/right_wheel.dae
- link RL_calf: geometry collision cylinder length=0.12 radius=0.013; visual mesh filename=package://go2w_description/dae/calf.dae
- link RL_foot: geometry collision cylinder length=0.045 radius=0.086; visual mesh filename=package://go2w_description/dae/left_wheel.dae
- link RR_calf: geometry collision cylinder length=0.12 radius=0.013; visual mesh filename=package://go2w_description/dae/calf_mirror.dae
- link RR_foot: geometry collision cylinder length=0.045 radius=0.086; visual mesh filename=package://go2w_description/dae/right_wheel.dae
Joints:
- joint FL_foot_joint: limit effort=23.7 velocity=30.1 -> lower=-999999 upper=999999 effort=23.7 velocity=30.1
- joint FR_foot_joint: limit effort=23.7 velocity=30.1 -> lower=-999999 upper=999999 effort=23.7 velocity=30.1
- joint RL_foot_joint: limit effort=23.7 velocity=30.1 -> lower=-999999 upper=999999 effort=23.7 velocity=30.1
- joint RR_foot_joint: limit effort=23.7 velocity=30.1 -> lower=-999999 upper=999999 effort=23.7 velocity=30.1
