Commit message: fix: update Deeprobotics models

File: source/robot_lab/data/Robots/deeprobotics/x30_description/urdf/x30.urdf (robot description, URDF)
Before this commit: robot X30, 17 links, 16 joints
Links:
- link FL_HIP: geometry visual mesh filename=../meshes/fl_hip.STL
- link FL_SHANK: geometry collision cylinder length=0.22 radius=0.025; visual mesh filename=../meshes/fl_shank.STL
- link FL_THIGH: geometry collision cylinder length=0.25 radius=0.04; visual mesh filename=../meshes/fl_thigh.STL
- link FR_HIP: geometry visual mesh filename=../meshes/fr_hip.STL
- link FR_SHANK: geometry collision cylinder length=0.22 radius=0.025; visual mesh filename=../meshes/fr_shank.STL
- link FR_THIGH: geometry collision cylinder length=0.25 radius=0.04; visual mesh filename=../meshes/fr_thigh.STL
- link HL_HIP: geometry visual mesh filename=../meshes/hl_hip.STL
- link HL_SHANK: geometry collision cylinder length=0.22 radius=0.025; visual mesh filename=../meshes/hl_shank.STL
- link HL_THIGH: geometry collision cylinder length=0.25 radius=0.04; visual mesh filename=../meshes/hl_thigh.STL
- link HR_HIP: geometry visual mesh filename=../meshes/hr_hip.STL
- link HR_SHANK: geometry collision cylinder length=0.22 radius=0.025; visual mesh filename=../meshes/hr_shank.STL
- link HR_THIGH: geometry collision cylinder length=0.25 radius=0.04; visual mesh filename=../meshes/hr_thigh.STL
- link TORSO: geometry collision box size=0.46 0.26 0.18; visual mesh filename=../meshes/torso.STL
