Commit message: update urdf

File: source/robot_lab/data/Robots/unitree/go2w_description/urdf/go2w_description.urdf (robot description, URDF)
Before this commit: robot go2w_description, 33 links, 32 joints
Links:
- removed link FL_calflower
- removed link FL_calflower1
- removed link FR_calflower
- removed link FR_calflower1
- removed link RL_calflower
- removed link RL_calflower1
- removed link RR_calflower
- removed link RR_calflower1
- link FL_calf: geometry collision box size=0.026 0.026 0.25; visual mesh filename=package://go2w_description/meshes/calf.stl
- link FL_foot_motor: geometry 
- link FL_hip: geometry collision sphere radius=0.046; visual mesh filename=package://go2w_description/meshes/hip.dae
- link FR_calf: geometry collision box size=0.026 0.026 0.25; visual mesh filename=package://go2w_description/meshes/calf_mirror.stl
- link FR_foot_motor: geometry 
- link FR_hip: geometry collision sphere radius=0.046; visual mesh filename=package://go2w_description/meshes/hip.dae
- link Head_upper: geometry collision sphere radius=0.06
- link RL_calf: geometry collision box size=0.026 0.026 0.25; visual mesh filename=package://go2w_description/meshes/calf.stl
- link RL_foot_motor: geometry 
- link RL_hip: geometry collision sphere radius=0.046; visual mesh filename=package://go2w_description/meshes/hip.dae
- link RR_calf: geometry collision box size=0.026 0.026 0.25; visual mesh filename=package://go2w_description/meshes/calf_mirror.stl
- link RR_foot_motor: geometry 
- link RR_hip: geometry collision sphere radius=0.046; visual mesh filename=package://go2w_description/meshes/hip.dae
Joints:
- removed joint FL_calflower1_joint
- removed joint FL_calflower_joint
- removed joint FR_calflower1_joint
- removed joint FR_calflower_joint
- removed joint RL_calflower1_joint
- removed joint RL_calflower_joint
- removed joint RR_calflower1_joint
- removed joint RR_calflower_joint

Commit message: update go2w

File: source/robot_lab/data/Robots/unitree/go2w_description/urdf/go2w_description.urdf (robot description, URDF)
Before this commit: robot go2w_description, 25 links, 24 joints
Links:
- added link FL_calflower; collision box size=0.022 0.022 0.065
- added link FL_calflower1; collision box size=0.031 0.031 0.03
- added link FR_calflower; collision box size=0.022 0.022 0.065
- added link FR_calflower1; collision box size=0.031 0.031 0.03
- added link RL_calflower; collision box size=0.022 0.022 0.065
- added link RL_calflower1; collision box size=0.031 0.031 0.03
- added link RR_calflower; collision box size=0.022 0.022 0.065
- added link RR_calflower1; collision box size=0.031 0.031 0.03
- link FL_calf: geometry collision box size=0.026 0.026 0.12; visual mesh filename=package://go2w_description/meshes/calf.stl
- link FR_calf: geometry collision box size=0.026 0.026 0.12; visual mesh filename=package://go2w_description/meshes/calf_mirror.stl
- link RL_calf: geometry collision box size=0.026 0.026 0.12; visual mesh filename=package://go2w_description/meshes/calf.stl
- link RR_calf: geometry collision box size=0.026 0.026 0.12; visual mesh filename=package://go2w_description/meshes/calf_mirror.stl
Joints:
- added joint FL_calflower1_joint: type fixed, parent FL_calflower, child FL_calflower1, origin xyz=-0.01 0 -0.04 rpy=0 0.48 0, axis 0 0 0
- added joint FL_calflower_joint: type fixed, parent FL_calf, child FL_calflower, origin xyz=0.020 0 -0.148 rpy=0 0.05 0, axis 0 0 0
- added joint FR_calflower1_joint: type fixed, parent FR_calflower, child FR_calflower1, origin xyz=-0.01 0 -0.04 rpy=0 0.48 0, axis 0 0 0
- added joint FR_calflower_joint: type fixed, parent FR_calf, child FR_calflower, origin xyz=0.020 0 -0.148 rpy=0 0.05 0, axis 0 0 0
- added joint RL_calflower1_joint: type fixed, parent RL_calflower, child RL_calflower1, origin xyz=-0.01 0 -0.04 rpy=0 0.48 0, axis 0 0 0
- added joint RL_calflower_joint: type fixed, parent RL_calf, child RL_calflower, origin xyz=0.020 0 -0.148 rpy=0 0.05 0, axis 0 0 0
- added joint RR_calflower1_joint: type fixed, parent RR_calflower, child RR_calflower1, origin xyz=-0.01 0 -0.04 rpy=0 0.48 0, axis 0 0 0
- added joint RR_calflower_joint: type fixed, parent RR_calf, child RR_calflower, origin xyz=0.020 0 -0.148 rpy=0 0.05 0, axis 0 0 0
